File: GarageDoor/kicad/door.kicad_pcb (KiCad board)
At the start: 2 copper layers, 150 x 100 mm, 19 parts, among them P1 LED_CONN, P10 SENS_2_CONN, P11 SENS_3_CONN, P12 LIGHT_CONN, P13 AUX_CONN, P2 LSW_U_CONN, P3 LSW_L_CONN, P4 MDO_CONN, P5 MDC_CONN, P6 AR_HE_HC05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

Commit message: Kicad stuff.
Parts:
- R1, R2: value 10K -> 1K
Connections:
- P10 pad 4: Net-(P10-Pad4) -> (no net)
- P11 pad 4: Net-(P11-Pad4) -> (no net)
- P7 pad 4: Net-(P7-Pad4) -> (no net)
- UNO1 pad 3V3: Net-(UNO1-Pad3V3) -> (no net)
- UNO1 pad AD3: Net-(UNO1-PadAD3) -> (no net)
- UNO1 pad AD4: Net-(UNO1-PadAD4) -> (no net)
- UNO1 pad AD5: Net-(UNO1-PadAD5) -> (no net)
- UNO1 pad AREF: Net-(UNO1-PadAREF) -> (no net)
- UNO1 pad RST: Net-(UNO1-PadRST) -> (no net)
- UNO1 pad V_IN: Net-(UNO1-PadV_IN) -> (no net)
