File: GarageDoor/kicad/door.sch (KiCad schematic (older format))
At the start: 19 parts, among them P1 LED_CONN, P10 SENS_2_CONN, P11 SENS_3_CONN, P12 LIGHT_CONN, P13 AUX_CONN, P2 LSW_U_CONN, P3 LSW_L_CONN, P4 MDO_CONN, P5 MDC_CONN, P6 AR_HE_HC05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

Commit message: Kicad
Parts:
- R1, R2, R3, R4, R5: symbol R -> R-RESCUE-door
Changed lines of the file:
@@
 EESchema Schematic File Version 2
+LIBS:door-rescue
 LIBS:power
 LIBS:device
@@
 LIBS:memory
 LIBS:xilinx
-LIBS:special
 LIBS:microcontrollers
 LIBS:dsp
@@
 LIBS:contrib
 LIBS:valves
-LIBS:arduino
 LIBS:door-cache
 EELAYER 25 0
@@
 $EndDescr
 $Comp
-L R R1
+L R-RESCUE-door R1
 U 1 1 547A1702
 P 4800 3550
@@
 $EndComp
 $Comp
-L R R2
+L R-RESCUE-door R2
 U 1 1 547A1784
 P 4800 4150
@@
 $EndComp
 $Comp
-L R R3
+L R-RESCUE-door R3
 U 1 1 547A17B7
 P 4800 4700
@@
 $EndComp
 $Comp
-L R R4
+L R-RESCUE-door R4
 U 1 1 547A17D2
 P 4800 5350
@@
 $EndComp
 $Comp
-L GND #PWR01
+L GND-RESCUE-door #PWR01
 U 1 1 547A7C83
 P 5200 3550
@@
 $EndComp
 $Comp
-L GND #PWR02
+L GND-RESCUE-door #PWR02
 U 1 1 547A7CF0
 P 5200 4700
@@
 $EndComp
 $Comp
-L GND #PWR03
+L GND-RESCUE-door #PWR03
 U 1 1 547A7D04
 P 5200 5350
@@
 $EndComp
 $Comp
-L GND #PWR05
+L GND-RESCUE-door #PWR05
 U 1 1 54B2E75A
 P 5200 4150
@@
 $EndComp
 $Comp
-L R R5
+L R-RESCUE-door R5
 U 1 1 54B309D8
 P 4250 3150
@@
 $EndComp
 $Comp
-L GND #PWR06
+L GND-RESCUE-door #PWR06
 U 1 1 54C3AAEC
 P 1650 3900
@@
 LED
 $Comp
-L GND #PWR07
+L GND-RESCUE-door #PWR07
 U 1 1 54C3B7F1
 P 9600 1050
@@
 ManualDoorCloseSwitch
 $Comp
-L GND #PWR011
+L GND-RESCUE-door #PWR011
 U 1 1 54C3ED6A
 P 10050 4400
@@
 $EndComp
 $Comp
-L GND #PWR014
+L GND-RESCUE-door #PWR014
 U 1 1 55059BB9
 P 9500 5450
@@
 $EndComp
 $Comp
-L GND #PWR015
+L GND-RESCUE-door #PWR015
 U 1 1 5505AEC6
 P 6150 1550
@@
 $EndComp
 $Comp
-L GND #PWR018
+L GND-RESCUE-door #PWR018
 U 1 1 55055FAF
 P 2900 1750
@@
 NoConn ~ 9100 5250
 $Comp
-L GND #PWR020
+L GND-RESCUE-door #PWR020
 U 1 1 55058A6F
 P 4050 3800
@@
 $EndComp
 $Comp
-L GND #PWR022
+L GND-RESCUE-door #PWR022
 U 1 1 550D2697
 P 1450 5700
@@
 $EndComp
 $Comp
-L GND #PWR024
+L GND-RESCUE-door #PWR024
 U 1 1 550D3E09
 P 1500 6600
@@
 	4100 2100 4450 2100
 $Comp
-L GND #PWR025
+L GND-RESCUE-door #PWR025
 U 1 1 551FBB48
 P 4350 2400
@@
 	2500 2100 2850 2100
 $Comp
-L GND #PWR026
+L GND-RESCUE-door #PWR026
 U 1 1 551FC9C4
 P 2800 2350

Commit message: Kicad stuff.
Parts:
- R1, R2: value 10K -> 1K
Changed lines of the file:
@@
 P 4800 3550
 F 0 "R1" V 4880 3550 40  0000 C CNN
-F 1 "10K" V 4807 3551 40  0000 C CNN
+F 1 "1K" V 4807 3551 40  0000 C CNN
 F 2 "Discret:R3-LARGE_PADS" V 4730 3550 30  0001 C CNN
 F 3 "" H 4800 3550 30  0000 C CNN
@@
 P 4800 4150
 F 0 "R2" V 4880 4150 40  0000 C CNN
-F 1 "10K" V 4807 4151 40  0000 C CNN
+F 1 "1K" V 4807 4151 40  0000 C CNN
 F 2 "Discret:R3-LARGE_PADS" V 4730 4150 30  0001 C CNN
 F 3 "" H 4800 4150 30  0000 C CNN
